Commit message: update height

File: src/sentry_bot/description/gazebo_control.xacro (robot description, xacro)
@@ -1,25 +1,48 @@
 <?xml version="1.0"?>
 <robot xmlns:xacro="http://www.ros.org/wiki/xacro">
-    <gazebo reference="mid_left_wheel">
-        <mu1 value="0.001"/><mu2 value="0.001"/>
-    </gazebo>
-    <gazebo reference="mid_right_wheel">
-        <mu1 value="0.001"/><mu2 value="0.001"/>
-    </gazebo>
+    <ros2_control name="IgnitionSystem" type="system">
+        <hardware>
+            <plugin>ign_ros2_control/IgnitionSystem</plugin>
+        </hardware>
+        <joint name="front_left_wheel_joint">
+            <command_interface name="velocity"><dt>0.01</dt></command_interface>
+            <state_interface name="velocity"/><state_interface name="position"/>
+        </joint>
+        <joint name="mid_left_wheel_joint">
+            <command_interface name="velocity"><dt>0.01</dt></command_interface>
+            <state_interface name="velocity"/><state_interface name="position"/>
+        </joint>
+        <joint name="back_left_wheel_joint">
+            <command_interface name="velocity"><dt>0.01</dt></command_interface>
+            <state_interface name="velocity"/><state_interface name="position"/>
+        </joint>
+        <joint name="front_right_wheel_joint">
+            <command_interface name="velocity"><dt>0.01</dt></command_interface>
+            <state_interface name="velocity"/><state_interface name="position"/>
+        </joint>
+        <joint name="mid_right_wheel_joint">
+            <command_interface name="velocity"><dt>0.01</dt></command_interface>
+            <state_interface name="velocity"/><state_interface name="position"/>
+        </joint>
+        <joint name="back_right_wheel_joint">
+            <command_interface name="velocity"><dt>0.01</dt></command_interface>
+            <state_interface name="velocity"/><state_interface name="position"/>
+        </joint>
+        <joint name="camera_pan_joint">
+            <state_interface name="position"/>
+        </joint>
+        <joint name="camera_tilt_joint">
+            <state_interface name="position"/>
+        </joint>
+    </ros2_control>
+    <gazebo reference="mid_left_wheel"><mu1>1.0</mu1><mu2>1.0</mu2></gazebo>
+    <gazebo reference="mid_right_wheel"><mu1>1.0</mu1><mu2>1.0</mu2></gazebo>
+    <gazebo reference="front_left_wheel"><mu1>0.1</mu1><mu2>0.1</mu2></gazebo>
+    <gazebo reference="back_left_wheel"><mu1>0.1</mu1><mu2>0.1</mu2></gazebo>
+    <gazebo reference="front_right_wheel"><mu1>0.1</mu1><mu2>0.1</mu2></gazebo>
+    <gazebo reference="back_right_wheel"><mu1>0.1</mu1><mu2>0.1</mu2></gazebo>
     <gazebo>
-        <plugin filename="ign_ros2_control-system" name="ign_ros2_control::IgnitionROS2ControlPlugin">
+        <plugin filename="libign_ros2_control-system.so" name="ign_ros2_control::IgnitionROS2ControlPlugin">
             <parameters>$(find sentry_bot)/config/my_controllers.yaml</parameters>
-        </plugin>
-        <plugin filename="libignition-gazebo-diff-drive-system.so" name="ignition::gazebo::systems::DiffDrive">
-            <left_joint>front_left_wheel_joint</left_joint>
-            <left_joint>back_left_wheel_joint</left_joint>
-            <right_joint>front_right_wheel_joint</right_joint>
-            <right_joint>back_right_wheel_joint</right_joint>
-            <wheel_separation>0.23</wheel_separation>
-            <wheel_diameter>0.094</wheel_diameter>
-            <topic>cmd_vel</topic>
-            <odom_topic>odom</odom_topic>
-            <frame_id>odom</frame_id>
-            <child_frame_id>base_link</child_frame_id>
         </plugin>
     </gazebo>
@@ -39,7 +62,6 @@
                 </scan>
                 <range>
-                    <min>0.1</min>
-                    <max>12.0</max>
-                </resolution>
+                    <min>0.1</min><max>12.0</max><resolution>0.01</resolution>
+                </range>
             </ray>
             <always_on>1</always_on>
@@ -54,8 +76,5 @@
             <camera>
                 <horizontal_fov>1.089</horizontal_fov>
-                <image>
-                    <width>640</width>
-                    <height>480</height>
-                </image>
+                <image><width>640</width><height>480</height></image>
                 <clip><near>0.05</near><far>8.0</far></clip>
             </camera>

File: src/sentry_bot/description/robot_core.xacro (robot description, xacro)
@@ -10,90 +10,95 @@
     <joint name="chassis_joint" type="fixed">
         <parent link="base_link"/><child link="chassis"/>
-        <origin xyz="-0.126 0 0"/>
+        <origin xyz="-0.126 0 0.04687"/>
     </joint>
     <link name="chassis">
-        <visual>
-            <origin xyz="0.126 0 0.046"/><geometry><box size="0.2524 0.2304 0.093"/></geometry>
-            <material name="black"/>
-        </visual>
-        <collision>
-            <origin xyz="0.126 0 0.046"/><geometry><box size="0.2524 0.2304 0.093"/></geometry>
-        </collision>
-        <xacro:inertial_box mass="2.5" x="0.2524" y="0.2304" z="0.093">
-            <origin xyz="0.126 0 0.046" rpy="0 0 0"/>
-        </xacro:inertial_box>
+        <visual><origin xyz="0.126 0 0.0225"/><geometry><box size="0.2524 0.2304 0.045"/></geometry><material name="black"/></visual>
+        <collision><origin xyz="0.126 0 0.0225"/><geometry><box size="0.2524 0.2304 0.045"/></geometry></collision>
+        <xacro:inertial_box mass="2.5" x="0.2524" y="0.2304" z="0.045"><origin xyz="0.126 0 0.0225"/></xacro:inertial_box>
     </link>
-    <joint name="upper_platform_joint" type="fixed">
-        <parent link="chassis"/><child link="upper_platform"/>
-        <origin xyz="0.063 0 0.093"/>
-    </joint>
+    <xacro:macro name="fender" params="prefix y_reflect">
+        <joint name="${prefix}_fender_joint" type="fixed">
+            <parent link="chassis"/>
+            <child link="${prefix}_fender"/>
+            <origin xyz="0.126 ${y_reflect * 0.1152} 0.045"/>
+        </joint>
+        <link name="${prefix}_fender">
+            <visual>
+                <origin xyz="0 ${y_reflect * 0.0125} -0.015"/><geometry><box size="0.28 0.025 0.03"/></geometry>
+                <material name="black"/>
+            </visual>
+        </link>
+    </xacro:macro>
+    <xacro:fender prefix="left" y_reflect="1"/><xacro:fender prefix="right" y_reflect="-1"/>
+    <xacro:macro name="pillar" params="prefix x_off y_off">
+        <joint name="${prefix}_pillar_joint" type="fixed"><parent link="chassis"/><child link="${prefix}_pillar"/><origin xyz="${0.126 + x_off} ${y_off} 0.045"/></joint>
+        <link name="${prefix}_pillar">
+            <visual><origin xyz="0 0 0.0225"/><geometry><cylinder radius="0.005" length="0.045"/></geometry><material name="grey"/></visual>
+        </link>
+    </xacro:macro>
+    <xacro:pillar prefix="fl" x_off="0.05" y_off="0.06"/><xacro:pillar prefix="fr" x_off="0.05" y_off="-0.06"/>
+    <xacro:pillar prefix="rl" x_off="-0.05" y_off="0.06"/><xacro:pillar prefix="rr" x_off="-0.05" y_off="-0.06"/>
+    <joint name="upper_platform_joint" type="fixed"><parent link="chassis"/><child link="upper_platform"/><origin xyz="0.126 0 0.090"/></joint>
     <link name="upper_platform">
-        <visual>
-            <origin xyz="0.063 0 0.0188"/><geometry><box size="0.126 0.120 0.0376"/></geometry>
-            <material name="black"/>
-        </visual>
-        <collision>
-            <origin xyz="0.063 0 0.0188"/><geometry><box size="0.126 0.120 0.0376"/></geometry>
-        </collision>
-        <xacro:inertial_box mass="0.5" x="0.126" y="0.120" z="0.0376">
-            <origin xyz="0.063 0 0.0188" rpy="0 0 0"/>
-        </xacro:inertial_box>
+        <visual><origin xyz="0 0 0.0225"/><geometry><box size="0.14 0.152 0.045"/></geometry><material name="black"/></visual>
+        <collision><origin xyz="0 0 0.0225"/><geometry><box size="0.14 0.152 0.045"/></geometry></collision>
+        <xacro:inertial_box mass="0.5" x="0.14" y="0.152" z="0.045"><origin xyz="0 0 0.0225"/></xacro:inertial_box>
     </link>
     <xacro:macro name="wheel" params="prefix x_off y_off">
-        <joint name="${prefix}_wheel_joint" type="continuous">
-            <parent link="base_link"/><child link="${prefix}_wheel"/>
-            <origin xyz="${x_off} ${y_off} 0" rpy="-${pi/2} 0 0"/><axis xyz="0 0 1"/>
-        </joint>
+        <joint name="${prefix}_wheel_joint" type="continuous"><parent link="base_link"/><child link="${prefix}_wheel"/><origin xyz="${x_off} ${y_off} 0.04687" rpy="-${pi/2} 0 0"/><axis xyz="0 0 1"/></joint>
         <link name="${prefix}_wheel">
             <visual><geometry><cylinder radius="0.04687" length="0.04"/></geometry><material name="grey"/></visual>
             <collision><geometry><cylinder radius="0.04687" length="0.04"/></geometry></collision>
-            <xacro:inertial_cylinder mass="0.2" length="0.04" radius="0.04687"><origin xyz="0 0 0" rpy="0 0 0"/></xacro:inertial_cylinder>
+            <xacro:inertial_cylinder mass="0.2" length="0.04" radius="0.04687"><origin xyz="0 0 0"/></xacro:inertial_cylinder>
         </link>
     </xacro:macro>
     <xacro:wheel prefix="front_left" x_off="0.10" y_off="0.115"/><xacro:wheel prefix="mid_left" x_off="0.0" y_off="0.115"/><xacro:wheel prefix="back_left" x_off="-0.10" y_off="0.115"/>
     <xacro:wheel prefix="front_right" x_off="0.10" y_off="-0.115"/><xacro:wheel prefix="mid_right" x_off="0.0" y_off="-0.115"/><xacro:wheel prefix="back_right" x_off="-0.10" y_off="-0.115"/>
-    <joint name="laser_joint" type="fixed">
-        <parent link="upper_platform"/><child link="laser_frame"/>
-        <origin xyz="0.1 0 0.0376" rpy="0 0 0"/>
-    </joint>
+    <joint name="laser_base_joint" type="fixed"><parent link="upper_platform"/><child link="laser_base"/><origin xyz="0.025 0 0.045"/></joint>
+    <link name="laser_base">
+        <visual><origin xyz="0 0 0.01"/><geometry><box size="0.04 0.04 0.02"/></geometry><material name="grey"/></visual>
+    </link>
+    <joint name="laser_joint" type="fixed"><parent link="laser_base"/><child link="laser_frame"/><origin xyz="0 0 0.02"/></joint>
     <link name="laser_frame">
-        <visual><geometry><cylinder radius="0.03" length="0.04"/></geometry><material name="blue"/></visual>
-        <collision><geometry><cylinder radius="0.03" length="0.04"/></geometry></collision>
-        <xacro:inertial_cylinder mass="0.1" length="0.04" radius="0.03"><origin xyz="0 0 0"/></xacro:inertial_cylinder>
+        <visual><origin xyz="0 0 0.01"/><geometry><cylinder radius="0.02" length="0.02"/></geometry><material name="blue"/></visual>
+        <collision><origin xyz="0 0 0.01"/><geometry><cylinder radius="0.02" length="0.02"/></geometry></collision>
     </link>
-    <joint name="camera_neck_joint" type="fixed"><parent link="upper_platform"/><child link="camera_neck"/><origin xyz="0.04 0 0.0376"/></joint>
-    <link name="camera_neck">
-        <visual><origin xyz="0 0 0.027"/><geometry><cylinder radius="0.02" length="0.054"/></geometry><material name="black"/></visual>
-        <collision><origin xyz="0 0 0.027"/><geometry><cylinder radius="0.02" length="0.054"/></geometry></collision>
-        <xacro:inertial_cylinder mass="0.05" length="0.054" radius="0.02"><origin xyz="0 0 0.027"/></xacro:inertial_cylinder>
+    <joint name="camera_stand_joint" type="fixed"><parent link="upper_platform"/><child link="camera_stand"/><origin xyz="-0.02 0 0.045"/></joint>
+    <link name="camera_stand">
+        <visual>
+            <origin xyz="0 0 0.015"/> <geometry><box size="0.05 0.04 0.03"/></geometry>
+            <material name="black"/>
+        </visual>
     </link>
-    <joint name="camera_pan_joint" type="continuous"><parent link="camera_neck"/><child link="camera_pan_link"/><origin xyz="0 0 0.054"/><axis xyz="0 0 1"/></joint>
+    <joint name="camera_pan_joint" type="continuous"><parent link="camera_stand"/><child link="camera_pan_link"/><origin xyz="0 0 0.03"/><axis xyz="0 0 1"/></joint>
     <link name="camera_pan_link">
-        <visual><origin xyz="0 0 0.01"/><geometry><cylinder radius="0.025" length="0.02"/></geometry><material name="grey"/></visual>
-        <xacro:inertial_cylinder mass="0.02" length="0.02" radius="0.025"><origin xyz="0 0 0.01"/></xacro:inertial_cylinder>
+        <visual>
+            <origin xyz="0 0 0.04"/> <geometry><cylinder radius="0.015" length="0.08"/></geometry>
+            <material name="grey"/>
+        </visual>
     </link>
     <joint name="camera_tilt_joint" type="revolute">
-        <parent link="camera_pan_link"/><child link="camera_head"/>
-        <origin xyz="0 0 0.02"/><axis xyz="0 1 0"/>
+        <parent link="camera_pan_link"/>
+        <child link="camera_head"/>
+        <origin xyz="0 0 0.08"/> <axis xyz="0 1 0"/>
         <limit lower="-1.57" upper="1.57" effort="10" velocity="1.0"/>
     </joint>
     <link name="camera_head">
-        <visual><origin xyz="0.02 0 0"/><geometry><box size="0.06 0.05 0.04"/></geometry><material name="red"/></visual>
-        <collision><origin xyz="0.02 0 0"/><geometry><box size="0.06 0.05 0.04"/></geometry></collision>
-        <xacro:inertial_box mass="0.1" x="0.06" y="0.05" z="0.04"><origin xyz="0.02 0 0"/></xacro:inertial_box>
+        <visual>
+            <origin xyz="0 0 0.025"/> <geometry><box size="0.05 0.05 0.05"/></geometry>
+            <material name="red"/>
+        </visual>
+        <collision>
+            <origin xyz="0 0 0.025"/>
+            <geometry><box size="0.05 0.05 0.05"/></geometry>
+        </collision>
+        <xacro:inertial_box mass="0.1" x="0.05" y="0.05" z="0.05"><origin xyz="0 0 0.025"/></xacro:inertial_box>
     </link>
     <xacro:macro name="antenna" params="prefix y_off">
-        <joint name="${prefix}_antenna_joint" type="fixed">
-            <parent link="upper_platform"/>
-            <child link="${prefix}_antenna"/>
-            <origin xyz="-0.01 ${y_off} 0.0376" rpy="0 -0.1 0"/>
-        </joint>
+        <joint name="${prefix}_antenna_joint" type="fixed"><parent link="upper_platform"/><child link="${prefix}_antenna"/><origin xyz="-0.068 ${y_off} 0.045" rpy="0 -0.1 0"/></joint>
         <link name="${prefix}_antenna">
             <visual><origin xyz="0 0 0.075"/><geometry><cylinder radius="0.003" length="0.15"/></geometry><material name="green"/></visual>
-            <collision><origin xyz="0 0 0.075"/><geometry><cylinder radius="0.003" length="0.15"/></geometry></collision>
-            <xacro:inertial_cylinder mass="0.01" length="0.15" radius="0.003"><origin xyz="0 0 0.075" rpy="0 0 0"/></xacro:inertial_cylinder>
         </link>
     </xacro:macro>
-    <xacro:antenna prefix="left" y_off="0.05"/>
-    <xacro:antenna prefix="right" y_off="-0.05"/>
+    <xacro:antenna prefix="left" y_off="0.05"/><xacro:antenna prefix="right" y_off="-0.05"/>
 </robot>
