Commit message: rviz2

File: src/sentry_bot/description/robot_core.xacro (robot description, xacro)
@@ -1,27 +1,44 @@
 <?xml version="1.0"?>
 <robot xmlns:xacro="http://www.ros.org/wiki/xacro">
-    <material name="black"><color rgba="0.0 0.0 0.0 1.0"/></material>
-    <material name="grey"><color rgba="0.5 0.5 0.5 1.0"/></material>
-    <material name="blue"><color rgba="0.2 0.2 1.0 1.0"/></material>
-    <material name="red"><color rgba="1.0 0.0 0.0 1.0"/></material>
-    <material name="green"><color rgba="0.0 1.0 0.0 1.0"/></material>
+    <material name="black">
+        <color rgba="0.0 0.0 0.0 1.0"/>
+    </material>
+    <material name="grey">
+        <color rgba="0.5 0.5 0.5 1.0"/>
+    </material>
+    <material name="blue">
+        <color rgba="0.2 0.2 1.0 1.0"/>
+    </material>
+    <material name="red">
+        <color rgba="1.0 0.0 0.0 1.0"/>
+    </material>
+    <material name="green">
+        <color rgba="0.0 1.0 0.0 1.0"/>
+    </material>
     <link name="base_link"></link>
     <joint name="chassis_joint" type="fixed">
-        <parent link="base_link"/><child link="chassis"/>
+        <parent link="base_link"/>
+        <child link="chassis"/>
         <origin xyz="-0.126 0 0"/>
     </joint>
     <link name="chassis">
         <visual>
-            <origin xyz="0.126 0 0.046"/><geometry><box size="0.2524 0.2304 0.093"/></geometry>
+            <origin xyz="0.126 0 0.046"/>
+            <geometry>
+                <box size="0.2524 0.2304 0.093"/> </geometry>
             <material name="black"/>
         </visual>
     </link>
     <joint name="upper_platform_joint" type="fixed">
-        <parent link="chassis"/><child link="upper_platform"/>
+        <parent link="chassis"/>
+        <child link="upper_platform"/>
         <origin xyz="0.063 0 0.093"/>
     </joint>
     <link name="upper_platform">
         <visual>
-            <origin xyz="0.063 0 0.018"/><geometry><box size="0.126 0.120 0.037"/></geometry>
+            <origin xyz="0.063 0 0.018"/>
+            <geometry>
+                <box size="0.126 0.120 0.037"/>
+            </geometry>
             <material name="black"/>
         </visual>
@@ -29,29 +46,47 @@
     <xacro:macro name="wheel" params="prefix x_off y_off">
         <joint name="${prefix}_wheel_joint" type="continuous">
-            <parent link="base_link"/><child link="${prefix}_wheel"/>
-            <origin xyz="${x_off} ${y_off} 0" rpy="-${pi/2} 0 0"/><axis xyz="0 0 1"/>
+            <parent link="base_link"/>
+            <child link="${prefix}_wheel"/>
+            <origin xyz="${x_off} ${y_off} 0" rpy="-${pi/2} 0 0"/>
+            <axis xyz="0 0 1"/>
         </joint>
         <link name="${prefix}_wheel">
-            <visual><geometry><cylinder radius="0.04687" length="0.04"/></geometry>
-            <material name="grey"/></visual>
+            <visual>
+                <geometry>
+                    <cylinder radius="0.04687" length="0.04"/> </geometry>
+                <material name="grey"/>
+            </visual>
         </link>
     </xacro:macro>
-    <xacro:wheel prefix="front_left"  x_off="0.10" y_off="0.115" /><xacro:wheel prefix="mid_left" x_off="0.0" y_off="0.115" /><xacro:wheel prefix="back_left" x_off="-0.10" y_off="0.115" />
-    <xacro:wheel prefix="front_right" x_off="0.10" y_off="-0.115" /><xacro:wheel prefix="mid_right" x_off="0.0" y_off="-0.115" /><xacro:wheel prefix="back_right" x_off="-0.10" y_off="-0.115" />
+    <xacro:wheel prefix="front_left"  x_off="0.10" y_off="0.115" />
+    <xacro:wheel prefix="mid_left"    x_off="0.0"  y_off="0.115" />
+    <xacro:wheel prefix="back_left"   x_off="-0.10" y_off="0.115" />
+    <xacro:wheel prefix="front_right" x_off="0.10" y_off="-0.115" />
+    <xacro:wheel prefix="mid_right"   x_off="0.0"  y_off="-0.115" />
+    <xacro:wheel prefix="back_right"  x_off="-0.10" y_off="-0.115" />
     <joint name="laser_joint" type="fixed">
-        <parent link="upper_platform"/><child link="laser_frame"/>
+        <parent link="upper_platform"/>
+        <child link="laser_frame"/>
         <origin xyz="0.1 0 0.037" rpy="0 0 0"/>
     </joint>
     <link name="laser_frame">
-        <visual><geometry><cylinder radius="0.03" length="0.04"/></geometry>
-        <material name="blue"/></visual>
+        <visual>
+            <geometry>
+                <cylinder radius="0.03" length="0.04"/>
+            </geometry>
+            <material name="blue"/>
+        </visual>
     </link>
     <joint name="camera_joint" type="fixed">
-        <parent link="upper_platform"/><child link="camera_link"/>
+        <parent link="upper_platform"/>
+        <child link="camera_link"/>
         <origin xyz="0.04 0 0.037" rpy="0 0 0"/>
     </joint>
     <link name="camera_link">
         <visual>
-            <origin xyz="0 0 0.075"/><geometry><box size="0.045 0.045 0.15"/></geometry>
+            <origin xyz="0 0 0.075"/>
+            <geometry>
+                <box size="0.045 0.045 0.15"/>
+            </geometry>
             <material name="red"/>
         </visual>
@@ -59,12 +94,19 @@
     <xacro:macro name="antenna" params="prefix y_off yaw_angle">
         <joint name="${prefix}_antenna_joint" type="fixed">
-            <parent link="upper_platform"/><child link="${prefix}_antenna"/>
+            <parent link="upper_platform"/>
+            <child link="${prefix}_antenna"/>
             <origin xyz="-0.02 ${y_off} 0.037" rpy="0 -0.2 ${yaw_angle}"/>
         </joint>
         <link name="${prefix}_antenna">
-            <visual><origin xyz="0 0 0.06"/><geometry><cylinder radius="0.003" length="0.132"/></geometry>
-            <material name="green"/></visual>
+            <visual>
+                <origin xyz="0 0 0.06"/>
+                <geometry>
+                    <cylinder radius="0.003" length="0.132"/>
+                </geometry>
+                <material name="green"/>
+            </visual>
         </link>
     </xacro:macro>
-    <xacro:antenna prefix="left" y_off="0.05" yaw_angle="0.3"/><xacro:antenna prefix="right" y_off="-0.05" yaw_angle="-0.3"/>
+    <xacro:antenna prefix="left"  y_off="0.05"  yaw_angle="0.3"/>
+    <xacro:antenna prefix="right" y_off="-0.05" yaw_angle="-0.3"/>
 </robot>

Commit message: working gazebo

File: src/sentry_bot/description/robot_core.xacro (robot description, xacro)
@@ -73,9 +73,15 @@
     <joint name="camera_pan_joint" type="continuous"><parent link="camera_stand"/><child link="camera_pan_link"/><origin xyz="0 0 0.03"/><axis xyz="0 0 1"/></joint>
     <link name="camera_pan_link">
-        <visual>
-            <origin xyz="0 0 0.04"/> <geometry><cylinder radius="0.015" length="0.08"/></geometry>
-            <material name="grey"/>
-        </visual>
-    </link>
+            <visual>
+                <origin xyz="0 0 0.04"/> <geometry><cylinder radius="0.015" length="0.08"/></geometry>
+                <material name="grey"/>
+            </visual>
+            <collision>
+                <origin xyz="0 0 0.04"/> <geometry><cylinder radius="0.015" length="0.08"/></geometry>
+            </collision>
+            <xacro:inertial_cylinder mass="0.05" length="0.08" radius="0.015">
+                <origin xyz="0 0 0.04"/>
+            </xacro:inertial_cylinder>
+        </link>
     <joint name="camera_tilt_joint" type="revolute">
         <parent link="camera_pan_link"/>
